File: hardware/peripheral/p2sgr-001.brd (EAGLE design)
At the start: 18 x 23 mm, 7 parts

Commit message: First working model.
Parts:
- removed J21, J22, J23, J24: (no value), SparkFun-Connectors:JST-4-PTH-VERT
- added J31, J32, J33, J34: (no value), SparkFun-Connectors:JST-3-PTH-VERT
- moved LOGO1 1.00 mm to (8.00, 11.0)
Connections:
- net ANLG0: now also J31.1; no longer J21.2
- net ANLG1: now also J32.1; no longer J22.2
- net ANLG2: now also J33.1; no longer J23.2
- net ANLG3: now also J34.1; no longer J24.2
- net DTCT0: no longer J21.1
- net DTCT1: no longer J22.1
- net DTCT2: no longer J23.1
- net DTCT3: no longer J24.1
- net GND: now also J31.2, J32.2, J33.2, J34.2; no longer J21.4, J22.4, J23.4, J24.4
- net VCC: now also J31.3, J32.3, J33.3, J34.3; no longer J21.3, J22.3, J23.3, J24.3
Routing:
- net DTCT2: track 13.9 -> 0.00 mm
- net DTCT1: track 13.4 -> 0.00 mm
- net DTCT3: track 13.3 -> 0.00 mm
- net DTCT0: track 13.2 -> 0.00 mm
- net GND: track 31.1 -> 39.8 mm
- net VCC: track 42.2 -> 39.9 mm
- net ANLG2: track 8.33 -> 10.00 mm
- net ANLG3: track 8.34 -> 9.36 mm
- net ANLG1: track 8.35 -> 9.35 mm
- net ANLG0: track 8.36 -> 9.36 mm
Other:
- board text added: "SharpGear 0.0.1-X"
- board text removed: "GroveGear 0.0.1-X"
