File: hardware/peripheral/p2sgr-001.sch (EAGLE design)
At the start: 7 parts

Commit message: First working model.
Parts:
- removed J21, J22, J23, J24: (no value), SparkFun-Connectors:CONN_04JST-PTH-VERT
- added J31, J32, J33, J34: (no value), SparkFun-Connectors:CONN_03JST-PTH-VERT
Connections:
- net ANLG0: now also J31.1; no longer J21.2
- net ANLG1: now also J32.1; no longer J22.2
- net ANLG2: now also J33.1; no longer J23.2
- net ANLG3: now also J34.1; no longer J24.2
- net DTCT0: no longer J21.1
- net DTCT1: no longer J22.1
- net DTCT2: no longer J23.1
- net DTCT3: no longer J24.1
- net GND: now also J31.2, J32.2, J33.2, J34.2; no longer J21.4, J22.4, J23.4, J24.4
- net VCC: now also J31.3, J32.3, J33.3, J34.3; no longer J21.3, J22.3, J23.3, J24.3
Changed lines of the file:
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@@
 <part name="SUPPLY3" library="supply2" library_urn="urn:adsk.eagle:library:372" deviceset="VCC" device=""/>
 <part name="U$1" library="pineapple" deviceset="PINEAPPLE450_SILK" device=""/>
-<part name="J21" library="SparkFun-Connectors" library_urn="urn:adsk.eagle:library:513" deviceset="CONN_04" device="JST-PTH-VERT" package3d_urn="urn:adsk.eagle:package:38102/1"/>
-<part name="J22" library="SparkFun-Connectors" library_urn="urn:adsk.eagle:library:513" deviceset="CONN_04" device="JST-PTH-VERT" package3d_urn="urn:adsk.eagle:package:38102/1"/>
-<part name="J23" library="SparkFun-Connectors" library_urn="urn:adsk.eagle:library:513" deviceset="CONN_04" device="JST-PTH-VERT" package3d_urn="urn:adsk.eagle:package:38102/1"/>
-<part name="J24" library="SparkFun-Connectors" library_urn="urn:adsk.eagle:library:513" deviceset="CONN_04" device="JST-PTH-VERT" package3d_urn="urn:adsk.eagle:package:38102/1"/>
+<part name="J31" library="SparkFun-Connectors" library_urn="urn:adsk.eagle:library:513" deviceset="CONN_03" device="JST-PTH-VERT" package3d_urn="urn:adsk.eagle:package:38080/1"/>
+<part name="J32" library="SparkFun-Connectors" library_urn="urn:adsk.eagle:library:513" deviceset="CONN_03" device="JST-PTH-VERT" package3d_urn="urn:adsk.eagle:package:38080/1"/>
+<part name="J33" library="SparkFun-Connectors" library_urn="urn:adsk.eagle:library:513" deviceset="CONN_03" device="JST-PTH-VERT" package3d_urn="urn:adsk.eagle:package:38080/1"/>
+<part name="J34" library="SparkFun-Connectors" library_urn="urn:adsk.eagle:library:513" deviceset="CONN_03" device="JST-PTH-VERT" package3d_urn="urn:adsk.eagle:package:38080/1"/>
 </parts>
 <sheets>
@@
 </instance>
 <instance part="U$1" gate="G$1" x="241.3" y="142.24" smashed="yes"/>
-<instance part="J21" gate="G$1" x="48.26" y="121.92" smashed="yes">
-<attribute name="VALUE" x="43.18" y="114.554" size="1.778" layer="96" font="vector"/>
+<instance part="J31" gate="J$1" x="45.72" y="124.46" smashed="yes">
+<attribute name="VALUE" x="43.18" y="117.094" size="1.778" layer="96" font="vector"/>
 <attribute name="NAME" x="43.18" y="130.048" size="1.778" layer="95" font="vector"/>
 </instance>
-<instance part="J22" gate="G$1" x="48.26" y="104.14" smashed="yes">
-<attribute name="VALUE" x="43.18" y="96.774" size="1.778" layer="96" font="vector"/>
+<instance part="J32" gate="J$1" x="45.72" y="106.68" smashed="yes">
+<attribute name="VALUE" x="43.18" y="99.314" size="1.778" layer="96" font="vector"/>
 <attribute name="NAME" x="43.18" y="112.268" size="1.778" layer="95" font="vector"/>
 </instance>
-<instance part="J23" gate="G$1" x="48.26" y="86.36" smashed="yes">
-<attribute name="VALUE" x="43.18" y="78.994" size="1.778" layer="96" font="vector"/>
+<instance part="J33" gate="J$1" x="45.72" y="88.9" smashed="yes">
+<attribute name="VALUE" x="43.18" y="81.534" size="1.778" layer="96" font="vector"/>
 <attribute name="NAME" x="43.18" y="94.488" size="1.778" layer="95" font="vector"/>
 </instance>
-<instance part="J24" gate="G$1" x="48.26" y="68.58" smashed="yes">
-<attribute name="VALUE" x="43.18" y="61.214" size="1.778" layer="96" font="vector"/>
+<instance part="J34" gate="J$1" x="45.72" y="71.12" smashed="yes">
+<attribute name="VALUE" x="43.18" y="63.754" size="1.778" layer="96" font="vector"/>
 <attribute name="NAME" x="43.18" y="76.708" size="1.778" layer="95" font="vector"/>
 </instance>
@@
 </segment>
 <segment>
-<pinref part="J21" gate="G$1" pin="4"/>
-<wire x1="53.34" y1="127" x2="58.42" y2="127" width="0.1524" layer="91"/>
-<label x="58.42" y="127" size="0.8128" layer="95" xref="yes"/>
-</segment>
-<segment>
-<pinref part="J22" gate="G$1" pin="4"/>
-<wire x1="53.34" y1="109.22" x2="58.42" y2="109.22" width="0.1524" layer="91"/>
-<label x="58.42" y="109.22" size="0.8128" layer="95" xref="yes"/>
-</segment>
-<segment>
-<pinref part="J23" gate="G$1" pin="4"/>
-<wire x1="53.34" y1="91.44" x2="58.42" y2="91.44" width="0.1524" layer="91"/>
-<label x="58.42" y="91.44" size="0.8128" layer="95" xref="yes"/>
-</segment>
-<segment>
-<pinref part="J24" gate="G$1" pin="4"/>
-<wire x1="53.34" y1="73.66" x2="58.42" y2="73.66" width="0.1524" layer="91"/>
-<label x="58.42" y="73.66" size="0.8128" layer="95" xref="yes"/>
+<wire x1="53.34" y1="124.46" x2="58.42" y2="124.46" width="0.1524" layer="91"/>
+<label x="58.42" y="124.46" size="0.8128" layer="95" xref="yes"/>
+<pinref part="J31" gate="J$1" pin="2"/>
+</segment>
+<segment>
+<wire x1="53.34" y1="106.68" x2="58.42" y2="106.68" width="0.1524" layer="91"/>
+<label x="58.42" y="106.68" size="0.8128" layer="95" xref="yes"/>
+<pinref part="J32" gate="J$1" pin="2"/>
+</segment>
+<segment>
+<wire x1="53.34" y1="88.9" x2="58.42" y2="88.9" width="0.1524" layer="91"/>
+<label x="58.42" y="88.9" size="0.8128" layer="95" xref="yes"/>
+<pinref part="J33" gate="J$1" pin="2"/>
+</segment>
+<segment>
+<wire x1="53.34" y1="71.12" x2="58.42" y2="71.12" width="0.1524" layer="91"/>
+<label x="58.42" y="71.12" size="0.8128" layer="95" xref="yes"/>
+<pinref part="J34" gate="J$1" pin="2"/>
 </segment>
 </net>
@@
 <wire x1="116.84" y1="109.22" x2="132.08" y2="109.22" width="0.1524" layer="91"/>
 <label x="132.08" y="109.22" size="0.8128" layer="95" xref="yes"/>
-</segment>
-<segment>
-<pinref part="J21" gate="G$1" pin="1"/>
-<wire x1="53.34" y1="119.38" x2="58.42" y2="119.38" width="0.1524" layer="91"/>
-<label x="58.42" y="119.38" size="0.8128" layer="95" xref="yes"/>
 </segment>
 </net>
@@
 </segment>
 <segment>
-<pinref part="J21" gate="G$1" pin="3"/>
-<wire x1="53.34" y1="124.46" x2="58.42" y2="124.46" width="0.1524" layer="91"/>
-<label x="58.42" y="124.46" size="0.8128" layer="95" xref="yes"/>
-</segment>
-<segment>
-<pinref part="J22" gate="G$1" pin="3"/>
-<wire x1="53.34" y1="106.68" x2="58.42" y2="106.68" width="0.1524" layer="91"/>
-<label x="58.42" y="106.68" size="0.8128" layer="95" xref="yes"/>
-</segment>
-<segment>
-<pinref part="J23" gate="G$1" pin="3"/>
-<wire x1="53.34" y1="88.9" x2="58.42" y2="88.9" width="0.1524" layer="91"/>
-<label x="58.42" y="88.9" size="0.8128" layer="95" xref="yes"/>
-</segment>
-<segment>
-<pinref part="J24" gate="G$1" pin="3"/>
-<wire x1="53.34" y1="71.12" x2="58.42" y2="71.12" width="0.1524" layer="91"/>
-<label x="58.42" y="71.12" size="0.8128" layer="95" xref="yes"/>
+<wire x1="53.34" y1="127" x2="58.42" y2="127" width="0.1524" layer="91"/>
+<label x="58.42" y="127" size="0.8128" layer="95" xref="yes"/>
+<pinref part="J31" gate="J$1" pin="3"/>
+</segment>
+<segment>
+<wire x1="53.34" y1="109.22" x2="58.42" y2="109.22" width="0.1524" layer="91"/>
+<label x="58.42" y="109.22" size="0.8128" layer="95" xref="yes"/>
+<pinref part="J32" gate="J$1" pin="3"/>
+</segment>
+<segment>
+<wire x1="53.34" y1="91.44" x2="58.42" y2="91.44" width="0.1524" layer="91"/>
+<label x="58.42" y="91.44" size="0.8128" layer="95" xref="yes"/>
+<pinref part="J33" gate="J$1" pin="3"/>
+</segment>
+<segment>
+<wire x1="53.34" y1="73.66" x2="58.42" y2="73.66" width="0.1524" layer="91"/>
+<label x="58.42" y="73.66" size="0.8128" layer="95" xref="yes"/>
+<pinref part="J34" gate="J$1" pin="3"/>
 </segment>
 </net>
@@
 <label x="132.08" y="104.14" size="0.8128" layer="95" xref="yes"/>
 </segment>
-<segment>
-<pinref part="J22" gate="G$1" pin="1"/>
-<wire x1="53.34" y1="101.6" x2="58.42" y2="101.6" width="0.1524" layer="91"/>
-<label x="58.42" y="101.6" size="0.8128" layer="95" xref="yes"/>
-</segment>
 </net>
 <net name="DTCT2" class="0">
@@
 <label x="132.08" y="99.06" size="0.8128" layer="95" xref="yes"/>
 </segment>
-<segment>
-<pinref part="J23" gate="G$1" pin="1"/>
-<wire x1="53.34" y1="83.82" x2="58.42" y2="83.82" width="0.1524" layer="91"/>
-<label x="58.42" y="83.82" size="0.8128" layer="95" xref="yes"/>
-</segment>
 </net>
 <net name="DTCT3" class="0">
@@
 <label x="132.08" y="93.98" size="0.8128" layer="95" xref="yes"/>
 </segment>
-<segment>
-<pinref part="J24" gate="G$1" pin="1"/>
-<wire x1="53.34" y1="66.04" x2="58.42" y2="66.04" width="0.1524" layer="91"/>
-<label x="58.42" y="66.04" size="0.8128" layer="95" xref="yes"/>
-</segment>
 </net>
 <net name="ANLG0" class="0">
@@
 </segment>
 <segment>
-<pinref part="J21" gate="G$1" pin="2"/>
 <wire x1="53.34" y1="121.92" x2="58.42" y2="121.92" width="0.1524" layer="91"/>
 <label x="58.42" y="121.92" size="0.8128" layer="95" xref="yes"/>
+<pinref part="J31" gate="J$1" pin="1"/>
 </segment>
 </net>
@@
 </segment>
 <segment>
-<pinref part="J22" gate="G$1" pin="2"/>
 <wire x1="53.34" y1="104.14" x2="58.42" y2="104.14" width="0.1524" layer="91"/>
 <label x="58.42" y="104.14" size="0.8128" layer="95" xref="yes"/>
+<pinref part="J32" gate="J$1" pin="1"/>
 </segment>
 </net>
@@
 </segment>
 <segment>
-<pinref part="J24" gate="G$1" pin="2"/>
 <wire x1="53.34" y1="68.58" x2="58.42" y2="68.58" width="0.1524" layer="91"/>
 <label x="58.42" y="68.58" size="0.8128" layer="95" xref="yes"/>
+<pinref part="J34" gate="J$1" pin="1"/>
 </segment>
 </net>
@@
 </segment>
 <segment>
-<pinref part="J23" gate="G$1" pin="2"/>
 <wire x1="53.34" y1="86.36" x2="58.42" y2="86.36" width="0.1524" layer="91"/>
 <label x="58.42" y="86.36" size="0.8128" layer="95" xref="yes"/>
-</segment>
-</net>
+<pinref part="J33" gate="J$1" pin="1"/>
+</segment>
+</net>
